File: hardware/front_panel/front_panel.kicad_pcb (KiCad board)
At the start: 2 copper layers, 25 x 44 mm, 12 parts, among them M1 Dark gray, M2 Dark gray, M3 Dark gray, M4 Dark gray, M5 Dark gray, M6 Dark gray

Commit message: Rev. A finished
Parts:
- moved M8 24.5 mm to (122.5, 98.5)
- moved M7 13.5 mm to (102.5, 98.5)
- moved M10 0.50 mm to (122.5, 142.0)
- moved M9 0.50 mm to (102.5, 142.0)
Other:
- board size 25 x 44 mm -> 28 x 50.5 mm
- board text added: "Nordic Clicker front panel Rev: A"
Changed lines of the file:
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@@
 	(generator_version "8.0")
 	(general
-		(thickness 1.6)
+		(thickness 1)
 		(legacy_teardrops no)
 	)
@@
 	)
 	(setup
+		(stackup
+			(layer "F.SilkS"
+				(type "Top Silk Screen")
+				(color "White")
+			)
+			(layer "F.Paste"
+				(type "Top Solder Paste")
+			)
+			(layer "F.Mask"
+				(type "Top Solder Mask")
+				(color "Black")
+				(thickness 0.01)
+			)
+			(layer "F.Cu"
+				(type "copper")
+				(thickness 0.035)
+			)
+			(layer "dielectric 1"
+				(type "core")
+				(thickness 0.91)
+				(material "FR4")
+				(epsilon_r 4.5)
+				(loss_tangent 0.02)
+			)
+			(layer "B.Cu"
+				(type "copper")
+				(thickness 0.035)
+			)
+			(layer "B.Mask"
+				(type "Bottom Solder Mask")
+				(color "Black")
+				(thickness 0.01)
+			)
+			(layer "B.Paste"
+				(type "Bottom Solder Paste")
+			)
+			(layer "B.SilkS"
+				(type "Bottom Silk Screen")
+				(color "White")
+			)
+			(copper_finish "None")
+			(dielectric_constraints no)
+		)
 		(pad_to_mask_clearance 0)
 		(allow_soldermask_bridges_in_footprints no)
@@
 		(model "${KIPLM_DIR}/kicad_libs/3d_models/BTNK03.step"
 			(offset
-				(xyz -2.8 4.75 -2.6)
+				(xyz -2.8 4.75 -2)
 			)
 			(scale
@@
 		(model "${KIPLM_DIR}/kicad_libs/3d_models/BTNK03.step"
 			(offset
-				(xyz -2.8 4.75 -2.6)
+				(xyz -2.8 4.75 -2)
 			)
 			(scale
@@
 		(model "${KIPLM_DIR}/kicad_libs/3d_models/BTNK03.step"
 			(offset
-				(xyz -2.8 4.75 -2.6)
+				(xyz -2.8 4.75 -2)
 			)
 			(scale
@@
 		(model "${KIPLM_DIR}/kicad_libs/3d_models/BTNK03.step"
 			(offset
-				(xyz -2.8 4.75 -2.6)
+				(xyz -2.8 4.75 -2)
 			)
 			(scale
@@
 		(model "${KIPLM_DIR}/kicad_libs/3d_models/BTNK03.step"
 			(offset
-				(xyz -2.8 4.75 -2.6)
+				(xyz -2.8 4.75 -2)
 			)
 			(scale
@@
 		(model "${KIPLM_DIR}/kicad_libs/3d_models/BTNK03.step"
 			(offset
-				(xyz -2.8 4.75 -2.6)
+				(xyz -2.8 4.75 -2)
 			)
 			(scale
@@
 	(footprint "KiPLM_Footprints:Threaded_Insert_M2_3.0mm_SMT"
 		(layer "B.Cu")
-		(at 106 111.5 180)
+		(at 102.5 98.5 180)
 		(property "Reference" "M7"
 			(at 0 0.5 0)
@@
 	(footprint "KiPLM_Footprints:Threaded_Insert_M2_3.0mm_SMT"
 		(layer "B.Cu")
-		(at 122.5 141.5 180)
+		(at 122.5 142 180)
 		(property "Reference" "M10"
 			(at 0 0.5 0)
@@
 	(footprint "KiPLM_Footprints:Threaded_Insert_M2_3.0mm_SMT"
 		(layer "B.Cu")
-		(at 102.5 141.5 180)
+		(at 102.5 142 180)
 		(property "Reference" "M9"
 			(at 0 0.5 0)
@@
 	(footprint "KiPLM_Footprints:Threaded_Insert_M2_3.0mm_SMT"
 		(layer "B.Cu")
-		(at 122.5 123 180)
+		(at 122.5 98.5 180)
 		(property "Reference" "M8"
 			(at 0 0.5 0)
@@
 		)
 	)
-	(gr_arc
-		(start 101 144)
-		(mid 100.292893 143.707107)
-		(end 100 143)
+	(gr_line
+		(start 100.5 95)
+		(end 124.5 95)
 		(stroke
 			(width 0.05)
@@
 	)
 	(gr_arc
-		(start 100 101)
-		(mid 100.292893 100.292893)
-		(end 101 100)
+		(start 124.5 95)
+		(mid 125.914214 95.585786)
+		(end 126.5 97)
 		(stroke
 			(width 0.05)
@@
 	)
 	(gr_line
-		(start 124 144)
-		(end 101 144)
+		(start 98.5 143.5)
+		(end 98.5 97)
 		(stroke
 			(width 0.05)
@@
 		(layer "Edge.Cuts")
 	)
-	(gr_line
-		(start 125 101)
-		(end 125 143)
+	(gr_arc
+		(start 98.5 97)
+		(mid 99.085786 95.585786)
+		(end 100.5 95)
 		(stroke
 			(width 0.05)
@@
 	)
 	(gr_line
-		(start 100 143)
-		(end 100 101)
+		(start 124.5 145.5)
+		(end 100.5 145.5)
 		(stroke
 			(width 0.05)
@@
 	)
 	(gr_line
-		(start 101 100)
-		(end 124 100)
+		(start 126.5 97)
+		(end 126.5 143.5)
 		(stroke
 			(width 0.05)
@@
 	)
 	(gr_arc
-		(start 124 100)
-		(mid 124.707107 100.292893)
-		(end 125 101)
+		(start 126.5 143.5)
+		(mid 125.914214 144.914214)
+		(end 124.5 145.5)
 		(stroke
 			(width 0.05)
@@
 	)
 	(gr_arc
-		(start 125 143)
-		(mid 124.707107 143.707107)
-		(end 124 144)
+		(start 100.5 145.5)
+		(mid 99.085786 144.914214)
+		(end 98.5 143.5)
 		(stroke
 			(width 0.05)
@@
 		(layer "Edge.Cuts")
 	)
+	(gr_text "Nordic Clicker\nfront panel\nRev: A"
+		(at 119.2 143.9 0)
+		(layer "B.SilkS" knockout)
+		(effects
+			(font
+				(size 1.2 1.2)
+				(thickness 0.25)
+				(bold yes)
+			)
+			(justify left bottom mirror)
+		)
+	)
 	(gr_text "FEEDBACK"
-		(at 105.8 108.7035 0)
+		(at 106.1 108.7035 0)
 		(layer "F.SilkS")
 		(effects
@@
 	)
 	(gr_text "COMMS"
-		(at 105.8 104.2035 0)
+		(at 106.1 104.2035 0)
 		(layer "F.SilkS")
 		(effects
